File: PCBs/status_board.kicad_sch (KiCad schematic)
At the start: 21 parts, among them J1 Conn_01x03, J2 Conn_01x03, J3 Conn_01x02, J4 Conn_01x04, J5 Conn_01x04, J6 Conn_01x04, J7 Conn_01x07, J8 Conn_01x07, J9 Conn_01x04

Commit message: fix depth connector + minor tweaks
Parts:
- J9: footprint Connector_JST:JST_SH_BM04B-SRSS-TB_1x04-1MP_P1.00mm_Vertical -> Connector_Hirose:Hirose_DF13C_CL535-0404-8-51_1x04-1MP_P1.25mm_Vertical
Changed lines of the file:
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@@
 			)
 		)
-		(property "Footprint" "Connector_JST:JST_SH_BM04B-SRSS-TB_1x04-1MP_P1.00mm_Vertical"
+		(property "Footprint" "Connector_Hirose:Hirose_DF13C_CL535-0404-8-51_1x04-1MP_P1.25mm_Vertical"
 			(at 123.19 83.82 0)
 			(hide yes)
