File: PCBs/status_board.kicad_pcb (KiCad board)
At the start: 2 copper layers, 43.5 x 36.5 mm, 21 parts, among them J1 Conn_01x03, J2 Conn_01x03, J3 Conn_01x02, J4 Conn_01x04, J5 Conn_01x04, J6 Conn_01x04, J7 Conn_01x07, J8 Conn_01x07, J9 Conn_01x04

Commit message: Revised board design
Parts:
- added  : LOGO, LOGO, F.Cu at (174.0, 78.5)
- renumbered J1 to J1,S, J2 to J2,C, R1 to R1,10k, R2 to R2,2.2k, R3 to R3,4.7k, R4 to R4,4.7k, R5 to R5,330, R6 to R6,330
Routing:
- net GND: track 92.8 -> 31.4 mm
- net Net-(J1-Pin_3): track 92.1 -> 91.5 mm
- added copper zone on B.Cu, net GND
Other:
- board text added: "Battery Probes"
- board text added: "Depth"
- board text added: "E"
- board text added: "Extra GPIO"
- board text added: "Hall Effect"
- board text added: "S"
- board text added: "Status Board"
- board text added: "Status LEDs"
- board text added: "Voltage Readout"
- board text removed: "10k"
- board text removed: "2.2k"
