File: PCBs/status_board.kicad_pcb (KiCad board)
At the start: 2 copper layers, 43.5 x 36.5 mm, 22 parts, among them J1,S Conn_01x03, J2,C Conn_01x03, J3 Conn_01x02, J4 Conn_01x04, J5 Conn_01x04, J6 Conn_01x04, J7 Conn_01x07, J8 Conn_01x07, J9 Conn_01x04

Commit message: fix depth connector + minor tweaks
Parts:
- J9: footprint Connector_JST:JST_SH_BM04B-SRSS-TB_1x04-1MP_P1.00mm_Vertical -> Connector_Hirose:Hirose_DF13C_CL535-0404-8-51_1x04-1MP_P1.25mm_Vertical
- moved J6 0.88 mm to (151.0, 73.0)
- moved H1 0.71 mm to (140.5, 72.0)
- moved J4 0.71 mm to (142.6, 85.5)
- moved J2 0.62 mm to (161.0, 73.0)
- moved J9 0.58 mm to (142.6, 78.2)
- moved H2 0.50 mm to (177.5, 72.0)
- moved H3 0.50 mm to (140.5, 102.0)
- renumbered J1,S to J1, J2,C to J2, R1,10k to R1, R2,2.2k to R2, R3,4.7k to R3, R4,4.7k to R4, R5,330 to R5, R6,330 to R6
Routing:
- net GND: track 31.4 -> 34.4 mm
- net Net-(J4-Pin_3): track 16.8 -> 19.7 mm
- net Net-(J4-Pin_2): track 20.7 -> 23.1 mm
- net Net-(J1-Pin_3): track 91.5 -> 93.7 mm
- net Net-(J6-Pin_2): track 5.21 -> 5.86 mm
Other:
- board size 43.5 x 36.5 mm -> 44 x 37 mm

Commit message: minor adjustments to depth conn
Parts:
- moved R3,4.7k 3.00 mm to (141.5, 90.2)
- moved R4,4.7k 3.00 mm to (144.5, 97.8)
- moved J9 0.75 mm to (142.6, 79.0), turned to 180 degrees
- turned J4 to 180 degrees
- renumbered R1 to R1,10k, R2 to R2,2.2k, R3 to R3,4.7k, R4 to R4,4.7k, R5 to R5,330, R6 to R6,330
Routing:
- net GND: track 34.4 -> 26.4 mm
- net Net-(J1-Pin_3): track 93.7 -> 100.5 mm
- net Net-(J4-Pin_2): track 23.1 -> 17.1 mm
- net Net-(J4-Pin_3): track 19.7 -> 24.9 mm
- net Net-(J6-Pin_1): track 24.3 -> 24.9 mm
